File: Avionics sensors.kicad_pcb (KiCad board)
At the start: 2 copper layers, 12 parts, among them U1 STM32L151CCTx, U2 MPU-6000

Commit message: Add files via upload
Parts:
- removed C6: 2.2nF, Capacitor_SMD:C_0805_2012Metric_Pad1.15x1.40mm_HandSolder
- added 2.2nF C6: 2.2nF, Capacitor_SMD:C_0603_1608Metric, F.Cu at (159.9, 84.9)
- 0.1uF C4: renamed from C4
- 0.1uF C5: renamed from C5
- 100nF C2: renamed from C-Ceramic2
- 100nF C3: renamed from C-Ceramic1
- 10uF Aluminum C: renamed from C-Aluminum1
- Terminal Block: renamed from REF**; value TerminalBlock_Phoenix_MKDS-1,5-2_1x02_P5.00mm_Horizontal -> TerminalBlock_Phoenix_MKDS-1,5-2_1x02
- renumbered Accelerometer1 to Accelerometer, U2 to IMU, REF** to Pins, PressureSensor1 to PressureSensor
Routing:
- net GND: track 122.5 -> 121.8 mm
